Commit message: moved table in kitchen.urdf

File: resources/kitchen.urdf (robot description, URDF)
Before this commit: robot iai_oven_area, 84 links, 83 joints
Joints:
- joint table_area_main_joint: origin xyz=-2.0 2.0 0 rpy=0 0 3.14159265359 -> xyz=-2.7 2.55 0 rpy=0 0 3.14159265359

Commit message: [CleanTheTableDemo] clean table ms2 demo, motion designator better error information, moveTorsoAction for parkArms added

File: resources/kitchen.urdf (robot description, URDF)
Before this commit: robot iai_oven_area, 84 links, 83 joints
Links:
- added link second_table_area, mass 1; collision mesh filename=package://iai_kitchen/meshes/misc/big_table_1.stl; visual mesh filename=package://iai_kitchen/meshes/misc/big_table_1.obj
Joints:
- added joint second_table_area_joint: type fixed, parent room_link, child second_table_area, origin xyz=-2.7 -0.6 0 rpy=0 0 3.14159265359
