Commit message: [robocup] some utils

File: resources/suturo_lab_version_15.urdf (robot description, URDF)
Before this commit: robot iai-kitchen, 129 links, 128 joints
Links:
- removed link kitchen_wall_1
- removed link kitchen_wall_2
- removed link kitchen_walls
- removed link wall_10_link
- removed link wall_11_link
- removed link wall_12_link
- removed link wall_13_link
- removed link wall_14_link
- removed link wall_15_link
- removed link wall_1_link
- removed link wall_2_link
- removed link wall_3_link
- removed link wall_4_link
- removed link wall_5_link
- removed link wall_9_link
Joints:
- removed joint wall_10_center_joint
- removed joint wall_11_center_joint
- removed joint wall_12_center_joint
- removed joint wall_13_center_joint
- removed joint wall_14_center_joint
- removed joint wall_15_center_joint
- removed joint wall_1_center_joint
- removed joint wall_1_joint
- removed joint wall_2_center_joint
- removed joint wall_2_joint
- removed joint wall_3_center_joint
- removed joint wall_4_center_joint
- removed joint wall_5_center_joint
- removed joint wall_9_center_joint
- removed joint walls_main_joint

Commit message: [Navigation/Receptionist] fixed some annoying stuff

File: resources/suturo_lab_version_15.urdf (robot description, URDF)
Before this commit: robot iai-kitchen, 129 links, 128 joints
Links:
- removed link arena_entry_exit:entry_exit:link
- removed link drawer_oven_right_board0_barrier_left_link
- removed link drawer_oven_right_board0_barrier_right_link
- removed link drawer_oven_right_board0_link
- removed link drawer_oven_right_board1_barrier_left_link
- removed link drawer_oven_right_board1_barrier_right_link
- removed link drawer_oven_right_board1_link
- removed link drawer_oven_right_board2_barrier_left_link
- removed link drawer_oven_right_board2_barrier_right_link
- removed link drawer_oven_right_board2_link
- removed link drawer_oven_right_board3_barrier_left_link
- removed link drawer_oven_right_board3_barrier_right_link
- removed link drawer_oven_right_board3_link
- removed link drawer_oven_right_front_link
- removed link fridge_area
- removed link fridge_area_footprint
- removed link fridge_area_lower_drawer_handle
- removed link fridge_area_lower_drawer_main
- removed link iai_fridge_door
- removed link iai_fridge_door_handle
- removed link iai_fridge_main
- removed link kitchen_island
- removed link kitchen_island_footprint
- removed link kitchen_island_left_lower_drawer_handle
- removed link kitchen_island_left_lower_drawer_main
- removed link kitchen_island_left_panel
- removed link kitchen_island_left_upper_drawer_handle
- removed link kitchen_island_left_upper_drawer_main
- removed link kitchen_island_middle_lower_drawer_handle
- removed link kitchen_island_middle_lower_drawer_main
- removed link kitchen_island_middle_panel
- removed link kitchen_island_middle_upper_drawer_handle
- removed link kitchen_island_middle_upper_drawer_main
- removed link kitchen_island_right_lower_drawer_handle
- removed link kitchen_island_right_lower_drawer_main
- removed link kitchen_island_right_panel
- removed link kitchen_island_right_upper_drawer_handle
- removed link kitchen_island_right_upper_drawer_main
- removed link kitchen_island_stove
- removed link kitchen_island_surface
- removed link kitchen_main
- removed link kitchen_wall_1
- removed link kitchen_wall_2
- removed link kitchen_walls
- removed link oven_area_area
- removed link oven_area_area_footprint
- removed link oven_area_area_left_drawer_handle
- removed link oven_area_area_left_drawer_main
- removed link oven_area_area_middle_lower_drawer_handle
- removed link oven_area_area_middle_lower_drawer_main
- removed link oven_area_area_middle_upper_drawer_handle
- removed link oven_area_area_middle_upper_drawer_main
- removed link oven_area_area_right_drawer_handle
- removed link oven_area_area_right_drawer_main
- removed link oven_area_oven_door
- removed link oven_area_oven_door_handle
- removed link oven_area_oven_knob_oven
- removed link oven_area_oven_knob_stove_1
- removed link oven_area_oven_knob_stove_2
- removed link oven_area_oven_knob_stove_3
- removed link oven_area_oven_knob_stove_4
- removed link oven_area_oven_main
- removed link oven_area_oven_panel
- removed link sink_area
- removed link sink_area_footprint
- removed link sink_area_left_bottom_drawer_handle
- removed link sink_area_left_bottom_drawer_main
- removed link sink_area_left_middle_drawer_handle
- removed link sink_area_left_middle_drawer_main
- removed link sink_area_left_upper_drawer_handle
- removed link sink_area_left_upper_drawer_main
- removed link sink_area_right_panel
- removed link sink_area_sink
- removed link sink_area_surface
- removed link sink_area_trash_drawer_handle
- removed link sink_area_trash_drawer_main
- removed link wall_10_link
- removed link wall_11_link
- removed link wall_12_link
- removed link wall_13_link
- removed link wall_14_link
- removed link wall_15_link
- removed link wall_1_link
- removed link wall_2_link
- removed link wall_3_link
- removed link wall_4_link
- removed link wall_5_link
- removed link wall_9_link
- added link arena_entry:entry:link
- added link arena_exit:exit:link
- added link chair:chair:chair_backrest; collision box size=0.3 0.05 0.5; visual box size=0.3 0.05 0.5
- added link chair:chair:chair_center; collision box size=0.3 0.3 0.5; visual box size=0.3 0.3 0.5
- added link chair:chair:chair_front_edge_center
- added link chair:chair:chair_origin
- added link dining_room:dining_room:room_center_link; collision box size=5.25 2.7 0.01; visual box size=5.25 2.7 0.01
- added link dining_room_entry_exit:entry_exit:link
- added link dishwasher_main, mass 1.0
- added link dishwasher_tab
- added link dishwasher_table:d_table:table_center; collision box size=0.6 0.6 0.02; visual box size=0.6 0.6 0.02
- added link dishwasher_table:d_table:table_front_edge_center
- added link dishwasher_table:d_table:table_origin
- added link kitchen_island:kitchen_island:table_center; collision box size=0.796 -2.47 0.853; visual box size=0.796 -2.47 0.853
- added link kitchen_island:kitchen_island:table_front_edge_center
- added link kitchen_island:kitchen_island:table_origin
- added link oven_area:oven_area:table_center; collision box size=0.68 1.2 1.51; visual box size=0.68 1.2 1.51
- added link oven_area:oven_area:table_front_edge_center
- added link oven_area:oven_area:table_origin
- added link refrigerator:refrigerator:table_center; collision box size=0.68 0.595 1.51; visual box size=0.68 0.595 1.51
- added link refrigerator:refrigerator:table_front_edge_center
- added link refrigerator:refrigerator:table_origin
- added link shelf_hohc:shelf_hohc:shelf_back; collision box size=0.02 0.8 2.02; visual box size=0.02 0.8 2.02
- added link shelf_hohc:shelf_hohc:shelf_base_center
- added link shelf_hohc:shelf_hohc:shelf_center
- added link shelf_hohc:shelf_hohc:shelf_door_left; collision box size=0.02 0.38 0.97; visual box size=0.02 0.38 0.97
- added link shelf_hohc:shelf_hohc:shelf_door_left:handle; collision box size=0.02 0.015 0.015; visual box size=0.02 0.015 0.015
- added link shelf_hohc:shelf_hohc:shelf_door_right; collision box size=0.02 0.38 0.97; visual box size=0.02 0.38 0.97
- added link shelf_hohc:shelf_hohc:shelf_door_right:handle; collision box size=0.02 0.015 0.015; visual box size=0.02 0.015 0.015
- added link shelf_hohc:shelf_hohc:shelf_floor_0; collision box size=0.4 0.8 0.04; visual box size=0.4 0.8 0.04
- added link shelf_hohc:shelf_hohc:shelf_floor_1; collision box size=0.4 0.8 0.04; visual box size=0.4 0.8 0.04
- added link shelf_hohc:shelf_hohc:shelf_floor_2; collision box size=0.4 0.8 0.04; visual box size=0.4 0.8 0.04
- added link shelf_hohc:shelf_hohc:shelf_floor_3; collision box size=0.4 0.8 0.04; visual box size=0.4 0.8 0.04
- added link shelf_hohc:shelf_hohc:shelf_left_side; collision box size=0.4 0.02 2.02; visual box size=0.4 0.02 2.02
- added link shelf_hohc:shelf_hohc:shelf_origin
- added link shelf_hohc:shelf_hohc:shelf_right_side; collision box size=0.4 0.02 2.02; visual box size=0.4 0.02 2.02
- added link work_surface_left:work_surface_left:table_center; collision box size=0.68 0.82 0.84; visual box size=0.68 0.82 0.84
- added link work_surface_left:work_surface_left:table_front_edge_center
- added link work_surface_left:work_surface_left:table_origin
- added link work_surface_right:work_surface_right:table_center; collision box size=0.68 0.64 0.84; visual box size=0.68 0.64 0.84
- added link work_surface_right:work_surface_right:table_front_edge_center
- added link work_surface_right:work_surface_right:table_origin
- link arena:arena:room_center_link: geometry collision box size=5.2 9.1 0.01; visual box size=5.2 9.1 0.01
- link iai_kitchen:kitchen:room_center_link: geometry collision box size=5.25 3.0 0.01; visual box size=5.25 3.0 0.01
- link living_room:living_room:room_center_link: geometry collision box size=5.25 3.4 0.01; visual box size=5.25 3.4 0.01
Joints:
- removed joint drawer_oven_right_board0_barrier_left_joint
- removed joint drawer_oven_right_board0_barrier_right_joint
- removed joint drawer_oven_right_board0_joint
- removed joint drawer_oven_right_board1_barrier_left_joint
- removed joint drawer_oven_right_board1_barrier_right_joint
- removed joint drawer_oven_right_board1_joint
- removed joint drawer_oven_right_board2_barrier_left_joint
- removed joint drawer_oven_right_board2_barrier_right_joint
- removed joint drawer_oven_right_board2_joint
- removed joint drawer_oven_right_board3_barrier_left_joint
- removed joint drawer_oven_right_board3_barrier_right_joint
- removed joint drawer_oven_right_board3_joint
- removed joint drawer_oven_right_front_joint
- removed joint fridge_area_footprint_joint
- removed joint fridge_area_lower_drawer_handle_joint
- removed joint fridge_area_lower_drawer_main_joint
- removed joint fridge_area_main_joint
- removed joint iai_fridge_door_handle_joint
- removed joint iai_fridge_door_joint
- removed joint iai_fridge_main_joint
- removed joint kitchen_island_footprint_joint
- removed joint kitchen_island_joint
- removed joint kitchen_island_left_lower_drawer_handle_joint
- removed joint kitchen_island_left_lower_drawer_main_joint
- removed joint kitchen_island_left_panel_joint
- removed joint kitchen_island_left_upper_drawer_handle_joint
- removed joint kitchen_island_left_upper_drawer_main_joint
- removed joint kitchen_island_middle_lower_drawer_handle_joint
- removed joint kitchen_island_middle_lower_drawer_main_joint
- removed joint kitchen_island_middle_panel_joint
- removed joint kitchen_island_middle_upper_drawer_handle_joint
- removed joint kitchen_island_middle_upper_drawer_main_joint
- removed joint kitchen_island_right_lower_drawer_handle_joint
- removed joint kitchen_island_right_lower_drawer_main_joint
- removed joint kitchen_island_right_panel_joint
- removed joint kitchen_island_right_upper_drawer_handle_joint
- removed joint kitchen_island_right_upper_drawer_main_joint
- removed joint kitchen_island_stove_joint
- removed joint kitchen_island_surface_joint
- removed joint kitchen_main
- removed joint oven_area_area_left_drawer_handle_joint
- removed joint oven_area_area_left_drawer_main_joint
- removed joint oven_area_area_middle_lower_drawer_handle_joint
- removed joint oven_area_area_middle_lower_drawer_main_joint
- removed joint oven_area_area_middle_upper_drawer_handle_joint
- removed joint oven_area_area_middle_upper_drawer_main_joint
- removed joint oven_area_area_right_drawer_handle_joint
- removed joint oven_area_area_right_drawer_joint
- removed joint oven_area_footprint_joint
- removed joint oven_area_main_joint
- removed joint oven_area_oven_door_handle_joint
- removed joint oven_area_oven_door_joint
- removed joint oven_area_oven_knob_oven_joint
- removed joint oven_area_oven_knob_stove_1_joint
- removed joint oven_area_oven_knob_stove_2_joint
- removed joint oven_area_oven_knob_stove_3_joint
- removed joint oven_area_oven_knob_stove_4_joint
- removed joint oven_area_oven_main_joint
- removed joint oven_area_oven_panel_joint
- removed joint room_arena_entry_exit:entry_exit:connection_joint
- removed joint sink_area_footprint_joint
- removed joint sink_area_left_bottom_drawer_handle_joint
- removed joint sink_area_left_bottom_drawer_main_joint
- removed joint sink_area_left_middle_drawer_handle_joint
- removed joint sink_area_left_middle_drawer_main_joint
- removed joint sink_area_left_upper_drawer_handle_joint
- removed joint sink_area_left_upper_drawer_main_joint
- removed joint sink_area_main_joint
- removed joint sink_area_right_panel_joint
- removed joint sink_area_sink_joint
- removed joint sink_area_surface_joint
- removed joint sink_area_trash_drawer_handle_joint
- removed joint sink_area_trash_drawer_main_joint
- removed joint wall_10_center_joint
- removed joint wall_11_center_joint
- removed joint wall_12_center_joint
- removed joint wall_13_center_joint
- removed joint wall_14_center_joint
- removed joint wall_15_center_joint
- removed joint wall_1_center_joint
- removed joint wall_1_joint
- removed joint wall_2_center_joint
- removed joint wall_2_joint
- removed joint wall_3_center_joint
- removed joint wall_4_center_joint
- removed joint wall_5_center_joint
- removed joint wall_9_center_joint
- removed joint walls_main_joint
- added joint chair:chair:center_joint: type fixed, parent chair:chair:chair_origin, child chair:chair:chair_center, origin xyz=0.0 0.0 0.25 rpy=0.0 0.0 0.0
- added joint chair:chair:chair_backrest_joint: type fixed, parent chair:chair:chair_center, child chair:chair:chair_backrest, origin xyz=0.0 -0.12 0.25 rpy=0.0 0.0 0.0
- added joint chair:chair:chair_front_edge_center_joint: type fixed, parent chair:chair:chair_origin, child chair:chair:chair_front_edge_center, origin xyz=0.0 0.15 0.5 rpy=0.0 0.0 0.0
- added joint chair:chair:chair_origin_joint: type fixed, parent urdf_offset, child chair:chair:chair_origin, origin xyz=2.8 1.3 0.0 rpy=0.0 0.0 0.0
- added joint dish_washer_table_center_joint: type fixed, parent dishwasher_table:d_table:table_origin, child dishwasher_table:d_table:table_front_edge_center, origin xyz=0.3 0.0 0.0 rpy=0.0 0.0 0.0
- added joint dish_washer_table_edge_joint: type fixed, parent dishwasher_table:d_table:table_origin, child dishwasher_table:d_table:table_center, origin xyz=0.0 0.0 0.0 rpy=0.0 0.0 0.0
- added joint dish_washer_table_main_joint: type fixed, parent sink_area_dish_washer_main, child dishwasher_table:d_table:table_origin, origin xyz=0.0 0.0 0.39 rpy=0.0 0.0 0.0
- added joint dishwasher_main: type fixed, parent urdf_offset, child dishwasher_main, origin xyz=1.86 -2.2 0.0 rpy=0.0 0.0 1.57
- added joint dishwasher_main_joint: type fixed, parent dishwasher_main, child sink_area_dish_washer_main, origin xyz=1.86 -2.2 0.0 rpy=0.0 0.0 1.57
- added joint dishwasher_tab_joint: type fixed, parent sink_area_dish_washer_door_handle, child dishwasher_tab, origin xyz=-0.1 0.1 0.15 rpy=0.0 0.0 0.0
- added joint kitchen_island:kitchen_island:center_joint: type fixed, parent kitchen_island:kitchen_island:table_origin, child kitchen_island:kitchen_island:table_center, origin xyz=0.398 -1.235 0.853 rpy=0.0 0.0 0.0
- added joint kitchen_island:kitchen_island:table_front_edge_center_joint: type fixed, parent kitchen_island:kitchen_island:table_origin, child kitchen_island:kitchen_island:table_front_edge_center, origin xyz=0.0 -1.235 0.853 rpy=0.0 0.0 0.0
- added joint kitchen_island:kitchen_island:table_origin_joint: type fixed, parent urdf_offset, child kitchen_island:kitchen_island:table_origin, origin xyz=3.0 0.134 0.0 rpy=0.0 0.0 1.57
- added joint oven_area:oven_area:center_joint: type fixed, parent oven_area:oven_area:table_origin, child oven_area:oven_area:table_center, origin xyz=0.34 0.6 1.51 rpy=0.0 0.0 0.0
- added joint oven_area:oven_area:table_front_edge_center_joint: type fixed, parent oven_area:oven_area:table_origin, child oven_area:oven_area:table_front_edge_center, origin xyz=0.0 0.6 1.51 rpy=0.0 0.0 0.0
- added joint oven_area:oven_area:table_origin_joint: type fixed, parent urdf_offset, child oven_area:oven_area:table_origin, origin xyz=3.77 -1.8 0.0 rpy=0.0 0.0 4.72
- added joint refrigerator:refrigerator:center_joint: type fixed, parent refrigerator:refrigerator:table_origin, child refrigerator:refrigerator:table_center, origin xyz=0.34 0.2975 1.51 rpy=0.0 0.0 0.0
- added joint refrigerator:refrigerator:table_front_edge_center_joint: type fixed, parent refrigerator:refrigerator:table_origin, child refrigerator:refrigerator:table_front_edge_center, origin xyz=0.0 0.2975 1.51 rpy=0.0 0.0 0.0
- added joint refrigerator:refrigerator:table_origin_joint: type fixed, parent urdf_offset, child refrigerator:refrigerator:table_origin, origin xyz=1.11 -1.84 0.0 rpy=0.0 0.0 4.72
- added joint room_arena_entry:entry:connection_joint: type fixed, parent arena:arena:room_center_link, child arena_entry:entry:link, origin xyz=-2.33 -2.05 0.0 rpy=0.0 0.0 0.0
- added joint room_arena_exit:exit:connection_joint: type fixed, parent arena:arena:room_center_link, child arena_exit:exit:link, origin xyz=-2.33 1.75 0.0 rpy=0.0 0.0 0.0
- added joint room_dining_room_entry_exit:entry_exit:connection_joint: type fixed, parent dining_room:dining_room:room_center_link, child dining_room_entry_exit:entry_exit:link, origin xyz=-0.7250000000000001 -1.35 0.0 rpy=0.0 0.0 0.0
- added joint shelf_hohc:shelf_hohc:shelf_back:joint: type fixed, parent shelf_hohc:shelf_hohc:shelf_origin, child shelf_hohc:shelf_hohc:shelf_back, origin xyz=0.4 0.4 1.01 rpy=0.0 0.0 0.0
- added joint shelf_hohc:shelf_hohc:shelf_base_center_joint: type fixed, parent shelf_hohc:shelf_hohc:shelf_origin, child shelf_hohc:shelf_hohc:shelf_base_center, origin xyz=0.2 0.4 0.0 rpy=0.0 0.0 0.0
- added joint shelf_hohc:shelf_hohc:shelf_center_joint: type fixed, parent shelf_hohc:shelf_hohc:shelf_origin, child shelf_hohc:shelf_hohc:shelf_center, origin xyz=0.2 0.4 1.01 rpy=0.0 0.0 0.0
- added joint shelf_hohc:shelf_hohc:shelf_door_left:handle_joint: type fixed, parent shelf_hohc:shelf_hohc:shelf_door_left, child shelf_hohc:shelf_hohc:shelf_door_left:handle, origin xyz=-0.03 -0.3575 0.09249999999999997 rpy=0.0 0.0 0.0, axis 0.0 0.0 1.0
- added joint shelf_hohc:shelf_hohc:shelf_door_left:joint: type revolute, parent shelf_hohc:shelf_hohc:shelf_left_side, child shelf_hohc:shelf_hohc:shelf_door_left, origin xyz=-0.19 -0.02 -0.48 rpy=0.0 0.0 0.0, axis 0.0 0.0 1.0, limit lower=-1.7 upper=0.0 effort=30.0 velocity=1.0
- added joint shelf_hohc:shelf_hohc:shelf_door_right:handle_joint: type fixed, parent shelf_hohc:shelf_hohc:shelf_door_right, child shelf_hohc:shelf_hohc:shelf_door_right:handle, origin xyz=-0.03 0.3575 0.09249999999999997 rpy=0.0 0.0 0.0, axis 0.0 0.0 1.0
- added joint shelf_hohc:shelf_hohc:shelf_door_right:joint: type revolute, parent shelf_hohc:shelf_hohc:shelf_right_side, child shelf_hohc:shelf_hohc:shelf_door_right, origin xyz=-0.19 0.02 -0.48 rpy=0.0 0.0 0.0, axis 0.0 0.0 1.0, limit lower=0.0 upper=1.7 effort=30.0 velocity=1.0
- added joint shelf_hohc:shelf_hohc:shelf_floor_0:joint: type fixed, parent shelf_hohc:shelf_hohc:shelf_base_center, child shelf_hohc:shelf_hohc:shelf_floor_0, origin xyz=0.0 0.0 0.1 rpy=0.0 0.0 0.0
- added joint shelf_hohc:shelf_hohc:shelf_floor_1:joint: type fixed, parent shelf_hohc:shelf_hohc:shelf_base_center, child shelf_hohc:shelf_hohc:shelf_floor_1, origin xyz=0.0 0.0 0.54 rpy=0.0 0.0 0.0
- added joint shelf_hohc:shelf_hohc:shelf_floor_2:joint: type fixed, parent shelf_hohc:shelf_hohc:shelf_base_center, child shelf_hohc:shelf_hohc:shelf_floor_2, origin xyz=0.0 0.0 1.055 rpy=0.0 0.0 0.0
- added joint shelf_hohc:shelf_hohc:shelf_floor_3:joint: type fixed, parent shelf_hohc:shelf_hohc:shelf_base_center, child shelf_hohc:shelf_hohc:shelf_floor_3, origin xyz=0.0 0.0 2.02 rpy=0.0 0.0 0.0
- added joint shelf_hohc:shelf_hohc:shelf_left_side:joint: type fixed, parent shelf_hohc:shelf_hohc:shelf_origin, child shelf_hohc:shelf_hohc:shelf_left_side, origin xyz=0.2 0.79 1.01 rpy=0.0 0.0 0.0
- added joint shelf_hohc:shelf_hohc:shelf_origin_joint: type fixed, parent urdf_offset, child shelf_hohc:shelf_hohc:shelf_origin, origin xyz=3.4 3.4 0.0 rpy=0.0 0.0 1.57
- added joint shelf_hohc:shelf_hohc:shelf_right_side:joint: type fixed, parent shelf_hohc:shelf_hohc:shelf_origin, child shelf_hohc:shelf_hohc:shelf_right_side, origin xyz=0.2 0.01 1.01 rpy=0.0 0.0 0.0
- added joint work_surface_left:work_surface_left:center_joint: type fixed, parent work_surface_left:work_surface_left:table_origin, child work_surface_left:work_surface_left:table_center, origin xyz=0.34 0.41 0.84 rpy=0.0 0.0 0.0
- added joint work_surface_left:work_surface_left:table_front_edge_center_joint: type fixed, parent work_surface_left:work_surface_left:table_origin, child work_surface_left:work_surface_left:table_front_edge_center, origin xyz=0.0 0.41 0.84 rpy=0.0 0.0 0.0
- added joint work_surface_left:work_surface_left:table_origin_joint: type fixed, parent urdf_offset, child work_surface_left:work_surface_left:table_origin, origin xyz=2.94 -1.84 0.0 rpy=0.0 0.0 4.72
- added joint work_surface_right:work_surface_right:center_joint: type fixed, parent work_surface_right:work_surface_right:table_origin, child work_surface_right:work_surface_right:table_center, origin xyz=0.34 0.32 0.84 rpy=0.0 0.0 0.0
- added joint work_surface_right:work_surface_right:table_front_edge_center_joint: type fixed, parent work_surface_right:work_surface_right:table_origin, child work_surface_right:work_surface_right:table_front_edge_center, origin xyz=0.0 0.32 0.84 rpy=0.0 0.0 0.0
- added joint work_surface_right:work_surface_right:table_origin_joint: type fixed, parent urdf_offset, child work_surface_right:work_surface_right:table_origin, origin xyz=1.705 -1.84 0.0 rpy=0.0 0.0 4.72
- added joint world_dining_room:dining_room:room_joint: type fixed, parent urdf_offset, child dining_room:dining_room:room_center_link, origin xyz=2.825 5.25 -0.05 rpy=0.0 0.0 0.0
- joint iai_kitchen:arena:door_handle_inside_joint: origin xyz=-0.07 0.0 0.065 rpy=0.0 0.0 1.5707963267948966 -> xyz=-0.02 0.0 0.055 rpy=0.0 0.0 1.5707963267948966
- joint living_room:arena:door_handle_inside_joint: origin xyz=-0.07 0.0 0.065 rpy=0.0 0.0 1.5707963267948966 -> xyz=-0.02 0.0 0.055 rpy=0.0 0.0 1.5707963267948966
- joint room_kitchen_entry_exit:entry_exit:connection_joint: origin xyz=-2.4 -0.66 0.0 rpy=0.0 0.0 0.0 -> xyz=-2.225 1.09 0.0 rpy=0.0 0.0 0.0
- joint room_living_room_entry_exit:entry_exit:connection_joint: origin xyz=-2.5300000000000002 -1.1400000000000001 0.0 rpy=0.0 0.0 0.0 -> xyz=-2.5650000000000004 1.6099999999999999 0.0 rpy=0.0 0.0 0.0
- joint sink_area_dish_washer_main_joint: origin xyz=0.01 0.1 0.044 rpy=0.0 0.0 0.0 -> xyz=0.08 -0.78 0.44 rpy=0.0 0.0 0.0; parent sink_area -> dishwasher_main
- joint world_arena:arena:room_joint: origin xyz=2.1 0.54 -0.05 rpy=0.0 0.0 0.0 -> xyz=3.0 2.05 -0.05 rpy=0.0 0.0 0.0
- joint world_iai_kitchen:kitchen:room_joint: origin xyz=3.0 0.75 -0.05 rpy=0.0 0.0 0.0 -> xyz=2.825 -1.0 -0.05 rpy=0.0 0.0 0.0
- joint world_living_room:living_room:room_joint: origin xyz=2.79 4.95 -0.05 rpy=0.0 0.0 0.0 -> xyz=2.825 2.2 -0.05 rpy=0.0 0.0 0.0
