Commit message: [robocup] recepetionist

File: resources/pre_robocup_5.urdf (robot description, URDF)
Before this commit: robot iai-kitchen, 129 links, 128 joints
Links:
- removed link wall_10_link
- removed link wall_11_link
- removed link wall_12_link
- removed link wall_13_link
- removed link wall_14_link
- removed link wall_15_link
- removed link wall_1_link
- removed link wall_2_link
- removed link wall_3_link
- removed link wall_4_link
- removed link wall_5_link
- removed link wall_9_link
Joints:
- removed joint wall_10_center_joint
- removed joint wall_11_center_joint
- removed joint wall_12_center_joint
- removed joint wall_13_center_joint
- removed joint wall_14_center_joint
- removed joint wall_15_center_joint
- removed joint wall_1_center_joint
- removed joint wall_2_center_joint
- removed joint wall_3_center_joint
- removed joint wall_4_center_joint
- removed joint wall_5_center_joint
- removed joint wall_9_center_joint
- joint iai_kitchen:arena:door_handle_inside_joint: origin xyz=-0.04 0.0 0.045 rpy=0.0 0.0 1.5707963267948966 -> xyz=-0.04 0.0 0.09 rpy=0.0 0.0 1.5707963267948966
- joint living_room:arena:door_handle_inside_joint: origin xyz=-0.04 0.0 0.045 rpy=0.0 0.0 1.5707963267948966 -> xyz=-0.04 0.0 0.09 rpy=0.0 0.0 1.5707963267948966
- joint living_room:arena:door_hinge_joint: origin xyz=0.28 3.37 1.04 rpy=0.0 0.0 0.0 -> xyz=0.23 3.3 1.04 rpy=0.0 0.0 0.0
