Commit message: fixing stuff

File: resources/after_robocup.urdf (robot description, URDF)
Before this commit: robot iai-kitchen, 110 links, 109 joints
Links:
- link arena:arena:room_center_link: mass 1.0 -> 0.0
- link coathanger:coathanger:coathanger_center: mass 1.0 -> 0.0
- link coffee_table:coffee_table:table_center: mass 1.0 -> 0.0
- link desk:desk:table_center: mass 1.0 -> 0.0
- link dinner_table:dinner_table:table_center: mass 1.0 -> 0.0
- link dishwasher_main: mass 1.0 -> 0.0
- link hallway:hallway:room_center_link: mass 1.0 -> 0.0
- link hallway_cabinet:hallway_cabinet:table_center: mass 1.0 -> 0.0
- link iai_kitchen:arena:door_center: mass 1.0 -> 0.0
- link iai_kitchen:arena:door_handle_inside: mass 1.0 -> 0.0
- link iai_kitchen:arena:door_handle_link: mass 1.0 -> 0.0
- link iai_kitchen:arena:door_handle_outside: mass 1.0 -> 0.0
- link iai_kitchen:arena:door_hinge: mass 1.0 -> 0.0
- link iai_kitchen:kitchen:room_center_link: mass 1.0 -> 0.0
- link kitchen_counter:kitchen_counter:table_center: mass 1.0 -> 0.0
- link lamp:lamp:lamp_center: mass 1.0 -> 0.0
- link living_room:living_room:room_center_link: mass 1.0 -> 0.0
- link office:arena:door_center: mass 1.0 -> 0.0
- link office:arena:door_handle_inside: mass 1.0 -> 0.0
- link office:arena:door_handle_link: mass 1.0 -> 0.0
- link office:arena:door_handle_outside: mass 1.0 -> 0.0
- link office:arena:door_hinge: mass 1.0 -> 0.0
- link office:office:room_center_link: mass 1.0 -> 0.0
- link shelf:shelf:shelf_back: mass 1.0 -> 0.0
- link shelf:shelf:shelf_floor_0: mass 1.0 -> 0.0
- link shelf:shelf:shelf_floor_1: mass 1.0 -> 0.0
- link shelf:shelf:shelf_floor_2: mass 1.0 -> 0.0
- link shelf:shelf:shelf_floor_3: mass 1.0 -> 0.0
- link shelf:shelf:shelf_left_side: mass 1.0 -> 0.0
- link shelf:shelf:shelf_right_side: mass 1.0 -> 0.0
- link shelf_hohc:kitchen_cabinet:shelf_back: mass 1.0 -> 0.0
- link shelf_hohc:kitchen_cabinet:shelf_door_left: mass 1.0 -> 0.0
- link shelf_hohc:kitchen_cabinet:shelf_door_left:handle: mass 1.0 -> 0.0
- link shelf_hohc:kitchen_cabinet:shelf_door_right: mass 1.0 -> 0.0
- link shelf_hohc:kitchen_cabinet:shelf_door_right:handle: mass 1.0 -> 0.0
- link shelf_hohc:kitchen_cabinet:shelf_floor_0: mass 1.0 -> 0.0
- link shelf_hohc:kitchen_cabinet:shelf_floor_1: mass 1.0 -> 0.0
- link shelf_hohc:kitchen_cabinet:shelf_floor_2: mass 1.0 -> 0.0
- link shelf_hohc:kitchen_cabinet:shelf_floor_3: mass 1.0 -> 0.0
- link shelf_hohc:kitchen_cabinet:shelf_floor_4: mass 1.0 -> 0.0
- link shelf_hohc:kitchen_cabinet:shelf_floor_5: mass 1.0 -> 0.0
- link shelf_hohc:kitchen_cabinet:shelf_floor_6: mass 1.0 -> 0.0
- link shelf_hohc:kitchen_cabinet:shelf_left_side: mass 1.0 -> 0.0
- link shelf_hohc:kitchen_cabinet:shelf_right_side: mass 1.0 -> 0.0
- link sink_area_dish_washer_door: mass 1.0 -> 0.0
- link sink_area_dish_washer_door_handle: mass 1.0 -> 0.0
- link sink_area_dish_washer_main: mass 1.0 -> 0.0
- link suturo_couch:couch:place_one: mass 1.0 -> 0.0
- link suturo_couch:couch:place_three: mass 1.0 -> 0.0
- link suturo_couch:couch:place_two: mass 1.0 -> 0.0
- link trashcan:trashcan:trashcan_center: mass 1.0 -> 0.0
- link tv_table:tv_table:table_center: mass 1.0 -> 0.0
- link wall_1_link: mass 1.0 -> 0.0
- link wall_2_link: mass 1.0 -> 0.0
- link wall_3_link: mass 1.0 -> 0.0
- link wall_4_link: mass 1.0 -> 0.0
- link wall_5_link: mass 1.0 -> 0.0
- link wall_6_link: mass 1.0 -> 0.0
- link wall_7_link: mass 1.0 -> 0.0
- link wall_8_link: mass 1.0 -> 0.0
