Commit message: [transporting] working on the semantic map

File: resources/apartment-small.urdf (robot description, URDF)
Before this commit: robot apartment, 97 links, 96 joints
Joints:
- joint table_area_main_joint: origin xyz=5 4 0 rpy=0 0 1.57 -> xyz=5 4 0.73 rpy=0 0 0

Commit message: [resources urdf] changed apartment small to know refrigerator

File: resources/apartment-small.urdf (robot description, URDF)
Before this commit: robot apartment, 98 links, 97 joints
Links:
- removed link cabinet3
- removed link cabinet3_door_bottom_left
- removed link cabinet3_door_bottom_out_fancy
- removed link cabinet3_door_top_left
- removed link cabinet3_door_top_out_fancy
- removed link handle_cab3_door_bottom
- removed link handle_cab3_door_top
- added link refrigerator; collision mesh filename=package://iai_apartment/meshes/cabinet03/IAICabinet3W60.obj; visual mesh filename=package://iai_apartment/meshes/cabinet03/IAICabinet3W60.dae
- added link refrigerator_door_bottom_handle; collision mesh filename=package://iai_apartment/meshes/handles/handle_horizontal.obj; visual mesh filename=package://iai_apartment/meshes/handles/handle_horizontal.dae
- added link refrigerator_door_bottom_left; collision mesh filename=package://iai_apartment/meshes/cabinet03/IAIDoorW60H80.obj; visual mesh filename=package://iai_apartment/meshes/cabinet03/IAIDoorW60H80.dae
- added link refrigerator_door_bottom_out_fancy
- added link refrigerator_door_top_handle; collision mesh filename=package://iai_apartment/meshes/handles/handle_horizontal.obj; visual mesh filename=package://iai_apartment/meshes/handles/handle_horizontal.dae
- added link refrigerator_door_top_left; collision mesh filename=package://iai_apartment/meshes/cabinet03/IAIDoorW60H133.obj; visual mesh filename=package://iai_apartment/meshes/cabinet03/IAIDoorW60H133.dae
- added link refrigerator_door_top_out_fancy
Joints:
- removed joint cabinet3_door_bottom_left_joint
- removed joint cabinet3_door_bottom_out_joint
- removed joint cabinet3_door_top_left_joint
- removed joint cabinet3_door_top_out_joint
- removed joint cabinet3_joint
- removed joint handle_cab3_door_bottom_joint
- removed joint handle_cab3_door_top_joint
- added joint refrigerator_door_bottom_handle_joint: type fixed, parent refrigerator_door_bottom_left, child refrigerator_door_bottom_handle, origin xyz=-0.036 -0.45 0.1 rpy=1.57 0 0
- added joint refrigerator_door_bottom_left_joint: type revolute, parent refrigerator_door_bottom_out_fancy, child refrigerator_door_bottom_left, axis 0 0 -1, limit lower=0.0 upper=1.5708 effort=1000.0 velocity=1.5708
- added joint refrigerator_door_bottom_out_joint: type prismatic, parent refrigerator, child refrigerator_door_bottom_out_fancy, origin xyz=0.39 -0.3 -0.5 rpy=0 0 3.14, axis -1 0 0, limit lower=0.0 upper=0.02 effort=1.0 velocity=1.5708, mimic joint=refrigerator_door_bottom_left_joint multiplier=0.01
- added joint refrigerator_door_top_handle_joint: type fixed, parent refrigerator_door_top_left, child refrigerator_door_top_handle, origin xyz=-0.036 -0.45 -0.65 rpy=1.57 0 0
- added joint refrigerator_door_top_left_joint: type revolute, parent refrigerator_door_top_out_fancy, child refrigerator_door_top_left, axis 0 0 -1, limit lower=0.0 upper=1.5708 effort=1000.0 velocity=1.5708
- added joint refrigerator_door_top_out_joint: type prismatic, parent refrigerator, child refrigerator_door_top_out_fancy, origin xyz=0.39 -0.3 0.5 rpy=0 0 3.14, axis -1 0 0, limit lower=0.0 upper=0.02 effort=1.0 velocity=1.5708, mimic joint=refrigerator_door_top_left_joint multiplier=0.01
- added joint refrigerator_joint: type fixed, parent side_A, child refrigerator, origin xyz=-0.273 1.022 1.07
