Commit message: [urdf] added floor

File: resources/robocane.urdf (robot description, URDF)
Before this commit: robot root, 89 links, 88 joints
Links:
- added link Floor_link, mass 0.0; collision box size=11 0.1 8.0; visual box size=10 0.2 10.1
Joints:
- added joint Floor_joint: type fixed, parent Environment, child Floor_link, origin xyz=5.5 3.0 0.0 rpy=1.570796012878418 0.0 0.0
