Commit message: [urdf_objects] added couch + shelf object

File: resources/suturo.urdf (robot description, URDF)
Before this commit: robot iai_suturo, 83 links, 82 joints
Links:
- added link shelf_billy:shelf_billy:shelf_back, mass 1.0; collision box size=0.02 0.8 2.02; visual box size=0.02 0.8 2.02
- added link shelf_billy:shelf_billy:shelf_base_center
- added link shelf_billy:shelf_billy:shelf_center
- added link shelf_billy:shelf_billy:shelf_door_left, mass 1.0; collision box size=0.02 0.4 0.97; visual box size=0.02 0.4 0.97
- added link shelf_billy:shelf_billy:shelf_door_left:handle, mass 1.0; collision cylinder length=0.02 radius=0.0075; visual cylinder length=0.02 radius=0.0075
- added link shelf_billy:shelf_billy:shelf_floor_0, mass 1.0; collision box size=0.39 0.8 0.04; visual box size=0.39 0.8 0.04
- added link shelf_billy:shelf_billy:shelf_floor_1, mass 1.0; collision box size=0.39 0.8 0.04; visual box size=0.39 0.8 0.04
- added link shelf_billy:shelf_billy:shelf_floor_2, mass 1.0; collision box size=0.39 0.8 0.04; visual box size=0.39 0.8 0.04
- added link shelf_billy:shelf_billy:shelf_floor_3, mass 1.0; collision box size=0.39 0.8 0.04; visual box size=0.39 0.8 0.04
- added link shelf_billy:shelf_billy:shelf_left_side, mass 1.0; collision box size=0.39 0.02 2.02; visual box size=0.39 0.02 2.02
- added link shelf_billy:shelf_billy:shelf_origin
- added link shelf_billy:shelf_billy:shelf_right_side, mass 1.0; collision box size=0.39 0.02 2.02; visual box size=0.39 0.02 2.02
- added link suturo_couch:couch:place_one, mass 1.0; collision box size=0.75 1.7 0.3; visual box size=0.75 1.7 0.3
- added link suturo_couch:couch:place_three, mass 1.0
- added link suturo_couch:couch:place_two, mass 1.0
Joints:
- added joint shelf_billy:shelf_billy:shelf_back:joint: type fixed, parent shelf_billy:shelf_billy:shelf_origin, child shelf_billy:shelf_billy:shelf_back, origin xyz=0.39 0.4 1.01 rpy=0.0 0.0 0.0
- added joint shelf_billy:shelf_billy:shelf_base_center_joint: type fixed, parent shelf_billy:shelf_billy:shelf_origin, child shelf_billy:shelf_billy:shelf_base_center, origin xyz=0.195 0.4 0.0 rpy=0.0 0.0 0.0
- added joint shelf_billy:shelf_billy:shelf_center_joint: type fixed, parent shelf_billy:shelf_billy:shelf_origin, child shelf_billy:shelf_billy:shelf_center, origin xyz=0.195 0.4 1.01 rpy=0.0 0.0 0.0
- added joint shelf_billy:shelf_billy:shelf_door_left:handle_joint: type fixed, parent shelf_billy:shelf_billy:shelf_door_left, child shelf_billy:shelf_billy:shelf_door_left:handle, origin xyz=-0.03 -0.3825 0.0075 rpy=0.0 1.5707963267948966 0.0, axis 0.0 0.0 1.0
- added joint shelf_billy:shelf_billy:shelf_door_left:joint: type revolute, parent shelf_billy:shelf_billy:shelf_left_side, child shelf_billy:shelf_billy:shelf_door_left, origin xyz=-0.215 0.0 -0.44 rpy=0.0 0.0 0.0, axis 0.0 0.0 1.0, limit lower=-1.7 upper=0.0 effort=30.0 velocity=1.0
- added joint shelf_billy:shelf_billy:shelf_floor_0:joint: type fixed, parent shelf_billy:shelf_billy:shelf_base_center, child shelf_billy:shelf_billy:shelf_floor_0, origin xyz=0.0 0.0 0.1 rpy=0.0 0.0 0.0
- added joint shelf_billy:shelf_billy:shelf_floor_1:joint: type fixed, parent shelf_billy:shelf_billy:shelf_base_center, child shelf_billy:shelf_billy:shelf_floor_1, origin xyz=0.0 0.0 0.54 rpy=0.0 0.0 0.0
- added joint shelf_billy:shelf_billy:shelf_floor_2:joint: type fixed, parent shelf_billy:shelf_billy:shelf_base_center, child shelf_billy:shelf_billy:shelf_floor_2, origin xyz=0.0 0.0 1.055 rpy=0.0 0.0 0.0
- added joint shelf_billy:shelf_billy:shelf_floor_3:joint: type fixed, parent shelf_billy:shelf_billy:shelf_base_center, child shelf_billy:shelf_billy:shelf_floor_3, origin xyz=0.0 0.0 2.02 rpy=0.0 0.0 0.0
- added joint shelf_billy:shelf_billy:shelf_left_side:joint: type fixed, parent shelf_billy:shelf_billy:shelf_origin, child shelf_billy:shelf_billy:shelf_left_side, origin xyz=0.195 0.79 1.01 rpy=0.0 0.0 0.0
- added joint shelf_billy:shelf_billy:shelf_origin_joint: type fixed, parent room_link, child shelf_billy:shelf_billy:shelf_origin, origin xyz=-5.3 2.5 0.0 rpy=0.0 0.0 1.57
- added joint shelf_billy:shelf_billy:shelf_right_side:joint: type fixed, parent shelf_billy:shelf_billy:shelf_origin, child shelf_billy:shelf_billy:shelf_right_side, origin xyz=0.195 0.01 1.01 rpy=0.0 0.0 0.0
- added joint suturo_couch:couch:couch_left_joint: type fixed, parent suturo_couch:couch:place_one, child suturo_couch:couch:place_two, origin xyz=0.0 -0.425 0.15 rpy=0.0 0.0 0.0
- added joint suturo_couch:couch:couch_origin_joint: type fixed, parent room_link, child suturo_couch:couch:place_one, origin xyz=-1.9 1.9 0.0 rpy=0.0 0.0 0.0
- added joint suturo_couch:couch:couch_right_joint: type fixed, parent suturo_couch:couch:place_one, child suturo_couch:couch:place_three, origin xyz=0.0 0.425 0.15 rpy=0.0 0.0 0.0

Commit message: [urdf_positions] moved table to correct position

File: resources/suturo.urdf (robot description, URDF)
Before this commit: robot iai_suturo, 98 links, 97 joints
Joints:
- joint table_area_main_joint: origin xyz=-3.3 0 0 rpy=0 0 0 -> xyz=-5.9 0.7 0 rpy=0 0 1.57

Commit message: [urdf_objects] colored couch and shelf. Also rotated and moved table to the other wall

File: resources/suturo.urdf (robot description, URDF)
Before this commit: robot iai_suturo, 98 links, 97 joints
Joints:
- joint table_area_main_joint: origin xyz=-5.9 0.7 0 rpy=0 0 1.57 -> xyz=-5.9 -0.5 0 rpy=0 0 1.57

Commit message: [urdf_objects] reduced unused urdf fragments of couch

File: resources/suturo.urdf (robot description, URDF)
Before this commit: robot iai_suturo, 98 links, 97 joints
Links:
- removed link suturo_couch:couch:place_one
- removed link suturo_couch:couch:place_three
- removed link suturo_couch:couch:place_two
- added link suturo_couch:couch:main, mass 1.0; collision box size=0.75 1.7 0.3; visual box size=0.75 1.7 0.3
Joints:
- removed joint suturo_couch:couch:couch_left_joint
- removed joint suturo_couch:couch:couch_right_joint
- joint suturo_couch:couch:couch_origin_joint: child suturo_couch:couch:place_one -> suturo_couch:couch:main

Commit message: [urdf_objects] added sofa.dae instead of plain box

File: resources/suturo.urdf (robot description, URDF)
Before this commit: robot iai_suturo, 96 links, 95 joints
Links:
- link suturo_couch:couch:main: geometry collision mesh filename=package://iai_apartment/meshes/visual/sofa.dae; visual mesh filename=package://iai_apartment/meshes/visual/sofa.dae
Joints:
- joint suturo_couch:couch:couch_origin_joint: origin xyz=-1.9 1.9 0.0 rpy=0.0 0.0 0.0 -> xyz=-1.9 1.9 0.0 rpy=0.0 0.0 -1.57

Commit message: [urdf_walls] reduced height of walls

File: resources/suturo.urdf (robot description, URDF)
Before this commit: robot iai_suturo, 96 links, 95 joints
Links:
- link kitchen_wall_1: geometry collision box size=1.1376 0.15 0.7; visual box size=1.1376 0.15 0.7
- link kitchen_wall_2: geometry collision box size=5.182 0.15 0.7; visual box size=5.182 0.15 0.7
- link kitchen_wall_3: geometry collision box size=8.901 0.15 0.7; visual box size=8.901 0.15 0.7

Commit message: [urdf_couch] moved couch to the shelf

File: resources/suturo.urdf (robot description, URDF)
Before this commit: robot iai_suturo, 96 links, 95 joints
Joints:
- joint suturo_couch:couch:couch_origin_joint: origin xyz=-1.9 1.9 0.0 rpy=0.0 0.0 -1.57 -> xyz=-3.9 2.55 0.0 rpy=0.0 0.0 0.0

Commit message: [suturo_urdf] added stools

File: resources/suturo.urdf (robot description, URDF)
Before this commit: robot iai_suturo, 96 links, 95 joints
Links:
- added link suturo_stool:stool1:main, mass 1.0; collision mesh filename=package://pycram/resources/stool.stl; visual mesh filename=package://pycram/resources/stool.stl
- added link suturo_stool:stool2:main, mass 1.0; collision mesh filename=package://pycram/resources/stool.stl; visual mesh filename=package://pycram/resources/stool.stl
Joints:
- added joint suturo_stool:stool1:stool_origin_joint: type fixed, parent room_link, child suturo_stool:stool1:main, origin xyz=-1.9 2.35 0.0 rpy=0.0 0.0 3.14
- added joint suturo_stool:stool2:stool_origin_joint: type fixed, parent room_link, child suturo_stool:stool2:main, origin xyz=-1.9 1.35 0.0 rpy=0.0 0.0 3.14

Commit message: [suturo_urdf] added couch table

File: resources/suturo.urdf (robot description, URDF)
Before this commit: robot iai_suturo, 98 links, 97 joints
Links:
- added link suturo_couch_table:couch_table:main, mass 1.0; collision mesh filename=package://iai_apartment/meshes/visual/coffee_table.dae; visual mesh filename=package://iai_apartment/meshes/visual/coffee_table.dae
Joints:
- added joint suturo_couch_table:couch_table:couch_table_origin_joint: type fixed, parent room_link, child suturo_couch_table:couch_table:main, origin xyz=-3.9 1.35 0.0 rpy=0.0 0.0 1.57
