Commit message: working on merging EVERYTHING big ass merge

File: resources/robots/hsrb.urdf (robot description, URDF)
Before this commit: robot hsrb, 49 links, 48 joints
Links:
- removed link base_b_bumper_link
- removed link base_f_bumper_link
- removed link hand_gripper_tool_frame
- link arm_flex_link: geometry collision mesh filename=package://hsr_meshes/meshes/arm_v0/arm_flex.collision.obj; visual mesh filename=package://hsr_meshes/meshes/arm_v0/arm_flex_light.obj
- link arm_lift_link: geometry collision mesh filename=package://hsr_meshes/meshes/arm_v0/shoulder.collision.obj; visual mesh filename=package://hsr_meshes/meshes/arm_v0/shoulder.obj
- link arm_roll_link: geometry collision mesh filename=package://hsr_meshes/meshes/arm_v0/arm_roll.collision.obj; visual mesh filename=package://hsr_meshes/meshes/arm_v0/arm_roll_light.obj
- link base_footprint: geometry collision box size=0.001 0.001 0.001
- link base_link: geometry collision mesh filename=package://hsr_meshes/meshes/base_v2/base.collision.obj; visual mesh filename=package://hsr_meshes/meshes/base_v2/base_light.obj
- link base_range_sensor_link: geometry collision mesh filename=package://hsr_meshes/meshes/sensors/laser.obj; visual mesh filename=package://hsr_meshes/meshes/sensors/laser.obj
- link hand_l_distal_link: geometry collision mesh filename=package://hsr_meshes/meshes/hand_v0/l_distal.obj; visual mesh filename=package://hsr_meshes/meshes/hand_v0/l_distal.obj
- link hand_l_spring_proximal_link: geometry collision mesh filename=package://hsr_meshes/meshes/hand_v0/l_proximal.obj; visual mesh filename=package://hsr_meshes/meshes/hand_v0/l_proximal.obj
- link hand_palm_link: geometry collision mesh filename=package://hsr_meshes/meshes/hand_v0/palm.obj; visual mesh filename=package://hsr_meshes/meshes/hand_v0/palm.obj
- link hand_r_distal_link: geometry collision mesh filename=package://hsr_meshes/meshes/hand_v0/r_distal.obj; visual mesh filename=package://hsr_meshes/meshes/hand_v0/r_distal.obj
- link hand_r_spring_proximal_link: geometry collision mesh filename=package://hsr_meshes/meshes/hand_v0/r_proximal.obj; visual mesh filename=package://hsr_meshes/meshes/hand_v0/r_proximal.obj
- link head_l_stereo_camera_link: geometry visual mesh filename=package://hsr_meshes/meshes/sensors/head_camera.obj
- link head_pan_link: geometry collision mesh filename=package://hsr_meshes/meshes/head_v1/head_pan.obj; visual mesh filename=package://hsr_meshes/meshes/head_v1/head_pan.obj
- link head_r_stereo_camera_link: geometry visual mesh filename=package://hsr_meshes/meshes/sensors/head_camera.obj
- link head_rgbd_sensor_link: geometry collision mesh filename=package://hsr_meshes/meshes/sensors/rgbd.obj; visual mesh filename=package://hsr_meshes/meshes/sensors/rgbd_light.obj
- link head_tilt_link: geometry collision mesh filename=package://hsr_meshes/meshes/head_v1/head.obj; collision mesh filename=package://hsr_meshes/meshes/head_v1/tablet.obj
- link torso_lift_link: geometry collision mesh filename=package://hsr_meshes/meshes/torso_v0/torso.collision.obj; visual mesh filename=package://hsr_meshes/meshes/torso_v0/torso_light.obj
- link wrist_flex_link: geometry collision cylinder length=0.04 radius=0.017; visual cylinder length=0.02 radius=0.017
- link wrist_roll_link: geometry collision mesh filename=package://hsr_meshes/meshes/wrist_v0/wrist_roll.collision.o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; visual mesh filename=package://hsr_meshes/meshes/wrist_v0/wrist_roll.obj
Joints:
- removed joint base_b_bumper_joint
- removed joint base_f_bumper_joint
- removed joint hand_gripper_tool_frame_joint
- joint arm_flex_joint: limit lower=-2.61 upper=-0.03 effort=100.0 velocity=1.2 -> lower=-2.62 upper=0.0 effort=100.0 velocity=1.2
- joint arm_lift_joint: limit lower=0.005 upper=0.67 effort=100.0 velocity=0.15 -> lower=0.0 upper=0.69 effort=100.0 velocity=0.2
- joint arm_roll_joint: limit lower=-1.95 upper=3.67 effort=100.0 velocity=2.0 -> lower=-2.09 upper=3.84 effort=100.0 velocity=2.0
- joint hand_camera_gazebo_frame_joint: origin xyz=0 0 0 rpy=1.570796326795 -1.570796326795 0 -> xyz=0 0 0 rpy=1.5707963268 -1.5707963268 0
- joint hand_l_finger_tip_frame_joint: origin xyz=0.01675 0.0193 0.0379 rpy=-1.570796326795 0.0 0.0 -> xyz=0.01675 0.0193 0.0379 rpy=-1.5707963268 0.0 0.0
- joint hand_l_finger_vacuum_frame_joint: origin xyz=0.00475 -0.011539 0.03322 rpy=0.7853981633975 0.0 0.0 -> xyz=0.00475 -0.011539 0.03322 rpy=0.785398163398 0.0 0.0
- joint hand_r_finger_tip_frame_joint: origin xyz=0.01675 -0.0193 0.0379 rpy=1.570796326795 0.0 0.0 -> xyz=0.01675 -0.0193 0.0379 rpy=1.5707963268 0.0 0.0
- joint head_center_camera_frame_joint: origin xyz=0.0195 0.0 0.061 rpy=-1.570796326795 0.0 -1.570796326795 -> xyz=0.0195 0.0 0.061 rpy=-1.5707963268 0.0 -1.5707963268
- joint head_center_camera_gazebo_frame_joint: origin xyz=0 0 0 rpy=1.570796326795 -1.570796326795 0.0 -> xyz=0 0 0 rpy=1.5707963268 -1.5707963268 0.0
- joint head_l_stereo_camera_gazebo_frame_joint: origin xyz=0 0 0 rpy=1.570796326795 -1.570796326795 0.0 -> xyz=0 0 0 rpy=1.5707963268 -1.5707963268 0.0
- joint head_l_stereo_camera_joint: origin xyz=0.02 0.07 0.061 rpy=-1.570796326795 0.0 -1.570796326795 -> xyz=0.02 0.07 0.061 rpy=-1.5707963268 0.0 -1.5707963268
- joint head_pan_joint: limit lower=-3.83 upper=1.74 effort=100.0 velocity=1.0 -> lower=-3.84 upper=1.75 effort=100.0 velocity=1.0
- joint head_r_stereo_camera_gazebo_frame_joint: origin xyz=0 0 0 rpy=1.570796326795 -1.570796326795 0.0 -> xyz=0 0 0 rpy=1.5707963268 -1.5707963268 0.0
- joint head_r_stereo_camera_joint: origin xyz=0.02 -0.07 0.061 rpy=-1.570796326795 0.0 -1.570796326795 -> xyz=0.02 -0.07 0.061 rpy=-1.5707963268 0.0 -1.5707963268
- joint head_rgbd_sensor_gazebo_frame_joint: origin xyz=0 0 0 rpy=1.570796326795 -1.570796326795 0.0 -> xyz=0 0 0 rpy=1.5707963268 -1.5707963268 0.0
- joint head_rgbd_sensor_joint: origin xyz=-0.079796 0.022 0.215172 rpy=-1.570796326795 0.0 -1.570796326795 -> xyz=-0.079796 0.022 0.215172 rpy=-1.5707963268 0.0 -1.5707963268
- joint head_tilt_joint: limit lower=-1.56 upper=0.47 effort=100.0 velocity=1.0 -> lower=-1.57 upper=0.52 effort=100.0 velocity=1.0
- joint torso_lift_joint: limit lower=0.0025 upper=0.335 effort=100.0 velocity=0.075 -> lower=0.0 upper=0.345 effort=100.0 velocity=0.1
- joint wrist_flex_joint: limit lower=-1.91 upper=1.21 effort=100.0 velocity=1.5 -> lower=-1.92 upper=1.22 effort=100.0 velocity=1.5
- joint wrist_ft_sensor_frame_joint: limit lower=0 upper=0 effort=100.0 velocity=1.5 -> (none); type revolute -> fixed
- joint wrist_roll_joint: limit lower=-1.91 upper=3.63 effort=100.0 velocity=1.5 -> lower=-1.92 upper=3.67 effort=100.0 velocity=1.5

File: resources/robots/pr2.urdf (robot description, URDF)
Before this commit: robot pr2, 88 links, 87 joints
Joints:
- joint torso_lift_joint: limit lower=0. upper=0.33 effort=1000 velocity=0.13 -> lower=0.0 upper=0.33 effort=10000 velocity=0.013
